Commit message: import matrices and a lot of examples and half-finished code

File: spryped rev03/urdf/spryped rev03.urdf (robot description, URDF)
Before this commit: robot spryped rev03, 9 links, 8 joints
Joints:
- joint 1: limit lower=0 upper=0 effort=0 velocity=0 -> lower=-1.57. upper=1.57. effort=0 velocity=1000; type continuous -> revolute
- joint 2: limit lower=0 upper=0 effort=0 velocity=0 -> lower=-1.57. upper=1.57. effort=0 velocity=1000; type continuous -> revolute
- joint 3: limit lower=0 upper=0 effort=0 velocity=0 -> lower=-1.57. upper=1.57. effort=0 velocity=1000; type continuous -> revolute
- joint 4: limit lower=0 upper=0 effort=0 velocity=0 -> lower=-1.57. upper=1.57. effort=0 velocity=1000; type continuous -> revolute
- joint 5: limit lower=0 upper=0 effort=0 velocity=0 -> lower=-1.57. upper=1.57. effort=0 velocity=1000; type continuous -> revolute
- joint 6: limit lower=0 upper=0 effort=0 velocity=0 -> lower=-1.57. upper=1.57. effort=0 velocity=1000; type continuous -> revolute
- joint 7: limit lower=0 upper=0 effort=0 velocity=0 -> lower=-1.57. upper=1.57. effort=0 velocity=1000; type continuous -> revolute
- joint 8: limit lower=0 upper=0 effort=0 velocity=0 -> lower=-1.57. upper=1.57. effort=0 velocity=1000; type continuous -> revolute
