Commit message: Troubleshooting wbc

File: res/spryped_urdf_rev06/urdf/spryped_urdf_rev06.urdf (robot description, URDF)
Before this commit: robot spryped_urdf_rev06, 9 links, 8 joints
Joints:
- joint 4: limit lower=-3.14 upper=3.14 effort=0 velocity=0 -> lower=-0.7 upper=0.9 effort=0 velocity=0
- joint 8: limit lower=-3.14 upper=3.14 effort=0 velocity=0 -> lower=-0.7 upper=0.9 effort=0 velocity=0
